Commit message: change robot finger and rope case. TODO: debug cloth case.

File: xarm/xarm6_with_gripper.urdf (robot description, URDF)
Before this commit: robot xarm6_with_gripper, 9 links, 8 joints
Links:
- link xarm_gripper_base_link: geometry collision mesh filename=xarm_gripper/meshes/stick.obj; visual mesh filename=xarm_gripper/meshes/stick.obj

Commit message: debug tshirt case.

File: xarm/xarm6_with_gripper.urdf (robot description, URDF)
Before this commit: robot xarm6_with_gripper, 9 links, 8 joints
Links:
- link xarm_gripper_base_link: geometry collision mesh filename=xarm_gripper/meshes/finger.obj; visual mesh filename=xarm_gripper/meshes/stick.obj
