Commit message: debugged sample action in env.

File: assets/xarm/xarm6_with_gripper_2.urdf (robot description, URDF)
Before this commit: robot xarm6_with_gripper, 15 links, 14 joints
Links:
- link left_finger: geometry collision mesh filename=xarm_gripper/meshes/left_finger.obj; visual mesh filename=xarm_gripper/meshes/left_finger.obj
- link right_finger: geometry collision mesh filename=xarm_gripper/meshes/right_finger.obj; visual mesh filename=xarm_gripper/meshes/right_finger.obj
- link xarm_gripper_base_link: geometry collision mesh filename=xarm_gripper/meshes/base_link.obj; visual mesh filename=xarm_gripper/meshes/base_link.obj
