Commit message: add more stickers; fixed the peneration problem for the rigid-granular case.

File: assets/xarm/xarm6_with_gripper.urdf (robot description, URDF)
Before this commit: robot xarm6_with_gripper, 9 links, 8 joints
Links:
- link xarm_gripper_base_link: geometry collision mesh filename=xarm_gripper/meshes/finger.obj; visual mesh filename=xarm_gripper/meshes/stick_2cm.obj

Commit message: adjust sample action for granular objects.

File: assets/xarm/xarm6_with_gripper.urdf (robot description, URDF)
Before this commit: robot xarm6_with_gripper, 9 links, 8 joints
Links:
- link xarm_gripper_base_link: geometry collision mesh filename=xarm_gripper/meshes/finger.obj; visual mesh filename=xarm_gripper/meshes/cynlinder.obj

Commit message: add rigid with different center of mass.

File: assets/xarm/xarm6_with_gripper.urdf (robot description, URDF)
Before this commit: robot xarm6_with_gripper, 9 links, 8 joints
Links:
- link xarm_gripper_base_link: geometry collision mesh filename=xarm_gripper/meshes/finger.obj; visual mesh filename=xarm_gripper/meshes/cylinder.obj

Commit message: change robot eef from pos to states.

File: assets/xarm/xarm6_with_gripper.urdf (robot description, URDF)
Before this commit: robot xarm6_with_gripper, 9 links, 8 joints
Links:
- link xarm_gripper_base_link: geometry collision mesh filename=xarm_gripper/meshes/cylinder.obj; visual mesh filename=xarm_gripper/meshes/cylinder.obj
